File: pcb_ruler.kicad_pcb (KiCad board)
At the start: 2 copper layers, 160 x 38 mm, 35 parts

Commit message: fix text
Other:
- board text added: "Elektrovägen 3 412 58 Göteborg Sweden"
- board text removed: "Elektrovägen 3 412 58 Gothenburg Sweden"
Changed lines of the file:
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@@
   (page A4)
   (layers
-    (0 F.Cu signal hide)
+    (0 F.Cu signal)
     (31 B.Cu signal)
     (32 B.Adhes user hide)
     (33 F.Adhes user hide)
     (34 B.Paste user)
-    (35 F.Paste user hide)
+    (35 F.Paste user)
     (36 B.SilkS user)
-    (37 F.SilkS user hide)
+    (37 F.SilkS user)
     (38 B.Mask user)
-    (39 F.Mask user hide)
+    (39 F.Mask user)
     (40 Dwgs.User user hide)
     (41 Cmts.User user)
@@
   (module prints:case_lab_logo_40x23mm (layer B.Cu)
     (at 237.9 107.5 180)
-    (fp_text reference G*** (at 0 0 180) (layer B.SilkS) hide
+    (fp_text reference G*** (at 0 0) (layer B.SilkS) hide
       (effects (font (size 1.524 1.524) (thickness 0.3)) (justify mirror))
     )
-    (fp_text value LOGO (at 0.75 0 180) (layer B.SilkS) hide
+    (fp_text value LOGO (at 0.75 0) (layer B.SilkS) hide
       (effects (font (size 1.524 1.524) (thickness 0.3)) (justify mirror))
     )
@@
       (xy 11.389199 0.028341) (xy 11.366571 -0.206) (xy 9.897 -0.225645) (xy 8.427428 -0.245291)
       (xy 8.427428 -1.403428) (xy 11.548 -1.403428) (xy 11.548 -1.911428) (xy 7.774286 -1.911428)
-      (xy 7.774286 1.792165) (xy 11.511714 1.753429)) (layer B.SilkS) (width 0.01))
+      (xy 7.774286 1.792165) (xy 11.511714 1.753429)) (layer B.Mask) (width 0.01))
     (fp_poly (pts (xy 7.048571 -1.911428) (xy 6.250286 -1.911428) (xy 6.250286 -1.258285) (xy 7.048571 -1.258285)
-      (xy 7.048571 -1.911428)) (layer B.SilkS) (width 0.01))
+      (xy 7.048571 -1.911428)) (layer B.Mask) (width 0.01))
     (fp_poly (pts (xy 5.597143 1.209143) (xy 3.933183 1.209143) (xy 3.386948 1.207879) (xy 2.967872 1.203319)
       (xy 2.657986 1.194311) (xy 2.439322 1.179702) (xy 2.293913 1.158339) (xy 2.203789 1.12907)
@@
       (xy 1.587571 1.42606) (xy 1.705815 1.533515) (xy 1.85416 1.618203) (xy 2.049898 1.682645)
       (xy 2.310321 1.729361) (xy 2.65272 1.76087) (xy 3.09439 1.779692) (xy 3.65262 1.788347)
-      (xy 4.083048 1.789715) (xy 5.597143 1.789715) (xy 5.597143 1.209143)) (layer B.SilkS) (width 0.01))
+      (xy 4.083048 1.789715) (xy 5.597143 1.789715) (xy 5.597143 1.209143)) (layer B.Mask) (width 0.01))
     (fp_poly (pts (xy 0.807428 -1.911428) (xy 0.009143 -1.911428) (xy 0.009143 -1.258285) (xy 0.807428 -1.258285)
-      (xy 0.807428 -1.911428)) (layer B.SilkS) (width 0.01))
+      (xy 0.807428 -1.911428)) (layer B.Mask) (width 0.01))
     (fp_poly (pts (xy -2.856599 1.746416) (xy -2.73108 1.662715) (xy -2.663053 1.570581) (xy -2.527041 1.373694)
       (xy -2.334343 1.088876) (xy -2.09626 0.732946) (xy -1.824093 0.322727) (xy -1.529141 -0.124961)
@@
       (xy -3.858441 0.87893) (xy -3.637611 1.198039) (xy -3.467198 1.433293) (xy -3.33747 1.597193)
       (xy -3.238694 1.702239) (xy -3.161135 1.760932) (xy -3.095061 1.785773) (xy -3.049407 1.789715)
-      (xy -2.856599 1.746416)) (layer B.SilkS) (width 0.01))
+      (xy -2.856599 1.746416)) (layer B.Mask) (width 0.01))
     (fp_poly (pts (xy -6.086857 -1.911428) (xy -6.885143 -1.911428) (xy -6.885143 -1.258285) (xy -6.086857 -1.258285)
-      (xy -6.086857 -1.911428)) (layer B.SilkS) (width 0.01))
+      (xy -6.086857 -1.911428)) (layer B.Mask) (width 0.01))
     (fp_poly (pts (xy -7.393143 1.209143) (xy -9.017114 1.209143) (xy -9.567467 1.207426) (xy -9.989053 1.201632)
       (xy -10.298212 1.1908) (xy -10.511288 1.173968) (xy -10.644621 1.150174) (xy -10.714553 1.118458)
@@
       (xy -11.240455 1.523729) (xy -11.041491 1.635386) (xy -10.758981 1.704979) (xy -10.378317 1.743802)
       (xy -9.884889 1.76315) (xy -9.264088 1.774319) (xy -9.116714 1.776674) (xy -7.393143 1.80481)
-      (xy -7.393143 1.209143)) (layer B.SilkS) (width 0.01))
+      (xy -7.393143 1.209143)) (layer B.Mask) (width 0.01))
   )
   (module Package_QFP:LQFP-32_5x5mm_P0.5mm (layer B.Cu)
@@
     (effects (font (size 0.9 0.9) (thickness 0.15)) (justify mirror))
   )
-  (gr_text www.caselabbet.se (at 237.8 129.5) (layer B.SilkS)
+  (gr_text www.caselabbet.se (at 237.8 129.5) (layer B.Mask)
     (effects (font (size 1.7 1.7) (thickness 0.2)) (justify mirror))
   )
@@
     (effects (font (size 0.8 0.8) (thickness 0.15)) (justify mirror))
   )
-  (gr_text "Elektrovägen 3\n412 58 Gothenburg\nSweden" (at 249.8 121) (layer B.SilkS)
+  (gr_text "Elektrovägen 3\n412 58 Göteborg\nSweden" (at 249.8 121) (layer B.Mask)
     (effects (font (size 1.8 1.8) (thickness 0.25)) (justify left mirror))
   )
